Commit message: aa

File: Proyecto/rover_rycsv/urdf/rover.urdf.xacro (robot description, xacro)
@@ -1,4 +1,4 @@
 <?xml version="1.0" encoding="utf-8"?>
-<robot name="rover_rycsv" xmlns:xacro="http://ros.org/wiki/xacro">
+<robot name="rover_gida" xmlns:xacro="http://ros.org/wiki/xacro">
   <xacro:arg name="imu_enable" default="true"/>
   <xacro:arg name="gps_enable" default="true"/>
@@ -29,5 +29,5 @@
       <geometry>
         <mesh
-          filename="package://rover_rycsv/meshes/Caja.STL" />
+          filename="package://rover_gida/meshes/Caja.STL" />
       </geometry>
       <material
@@ -81,5 +81,5 @@
       <geometry>
         <mesh
-          filename="package://rover_rycsv/meshes/Rocker_izq.STL" />
+          filename="package://rover_gida/meshes/Rocker_izq.STL" />
       </geometry>
       <material
@@ -135,5 +135,5 @@
       <geometry>
         <mesh
-          filename="package://rover_rycsv/meshes/Bogie_izq.STL" />
+          filename="package://rover_gida/meshes/Bogie_izq.STL" />
       </geometry>
       <material
@@ -189,5 +189,5 @@
       <geometry>
         <mesh
-          filename="package://rover_rycsv/meshes/Acople_1.STL" />
+          filename="package://rover_gida/meshes/Acople_1.STL" />
       </geometry>
       <material
@@ -243,5 +243,5 @@
       <geometry>
         <mesh
-          filename="package://rover_rycsv/meshes/Rueda_1.STL" />
+          filename="package://rover_gida/meshes/Rueda_1.STL" />
       </geometry>
       <material
@@ -257,5 +257,5 @@
       <geometry>
         <mesh
-          filename="package://rover_rycsv/meshes/Rueda_1.STL" />
+          filename="package://rover_gida/meshes/Rueda_1.STL" />
       </geometry>
     </collision>
@@ -299,5 +299,5 @@
       <geometry>
         <mesh
-          filename="package://rover_rycsv/meshes/Acople_2.STL" />
+          filename="package://rover_gida/meshes/Acople_2.STL" />
       </geometry>
       <material
@@ -351,5 +351,5 @@
       <geometry>
         <mesh
-          filename="package://rover_rycsv/meshes/Rueda_2.STL" />
+          filename="package://rover_gida/meshes/Rueda_2.STL" />
       </geometry>
       <material
@@ -365,5 +365,5 @@
       <geometry>
         <mesh
-          filename="package://rover_rycsv/meshes/Rueda_2.STL" />
+          filename="package://rover_gida/meshes/Rueda_2.STL" />
       </geometry>
     </collision>
@@ -407,5 +407,5 @@
       <geometry>
         <mesh
-          filename="package://rover_rycsv/meshes/Acople_3.STL" />
+          filename="package://rover_gida/meshes/Acople_3.STL" />
       </geometry>
       <material
@@ -461,5 +461,5 @@
       <geometry>
         <mesh
-          filename="package://rover_rycsv/meshes/Rueda_3.STL" />
+          filename="package://rover_gida/meshes/Rueda_3.STL" />
       </geometry>
       <material
@@ -475,5 +475,5 @@
       <geometry>
         <mesh
-          filename="package://rover_rycsv/meshes/Rueda_3.STL" />
+          filename="package://rover_gida/meshes/Rueda_3.STL" />
       </geometry>
     </collision>
@@ -517,5 +517,5 @@
       <geometry>
         <mesh
-          filename="package://rover_rycsv/meshes/Rocker_der.STL" />
+          filename="package://rover_gida/meshes/Rocker_der.STL" />
       </geometry>
       <material
@@ -571,5 +571,5 @@
       <geometry>
         <mesh
-          filename="package://rover_rycsv/meshes/Bogie_der.STL" />
+          filename="package://rover_gida/meshes/Bogie_der.STL" />
       </geometry>
       <material
@@ -625,5 +625,5 @@
       <geometry>
         <mesh
-          filename="package://rover_rycsv/meshes/Acople_4.STL" />
+          filename="package://rover_gida/meshes/Acople_4.STL" />
       </geometry>
       <material
@@ -679,5 +679,5 @@
       <geometry>
         <mesh
-          filename="package://rover_rycsv/meshes/Rueda_4.STL" />
+          filename="package://rover_gida/meshes/Rueda_4.STL" />
       </geometry>
       <material
@@ -693,5 +693,5 @@
       <geometry>
         <mesh
-          filename="package://rover_rycsv/meshes/Rueda_4.STL" />
+          filename="package://rover_gida/meshes/Rueda_4.STL" />
       </geometry>
     </collision>
@@ -735,5 +735,5 @@
       <geometry>
         <mesh
-          filename="package://rover_rycsv/meshes/Acople_5.STL" />
+          filename="package://rover_gida/meshes/Acople_5.STL" />
       </geometry>
       <material
@@ -787,5 +787,5 @@
       <geometry>
         <mesh
-          filename="package://rover_rycsv/meshes/Rueda_5.STL" />
+          filename="package://rover_gida/meshes/Rueda_5.STL" />
       </geometry>
       <material
@@ -801,5 +801,5 @@
       <geometry>
         <mesh
-          filename="package://rover_rycsv/meshes/Rueda_5.STL" />
+          filename="package://rover_gida/meshes/Rueda_5.STL" />
       </geometry>
     </collision>
@@ -843,5 +843,5 @@
       <geometry>
         <mesh
-          filename="package://rover_rycsv/meshes/Acople_6.STL" />
+          filename="package://rover_gida/meshes/Acople_6.STL" />
       </geometry>
       <material
@@ -897,5 +897,5 @@
       <geometry>
         <mesh
-          filename="package://rover_rycsv/meshes/Rueda_6.STL" />
+          filename="package://rover_gida/meshes/Rueda_6.STL" />
       </geometry>
       <material
@@ -911,5 +911,5 @@
       <geometry>
         <mesh
-          filename="package://rover_rycsv/meshes/Rueda_6.STL" />
+          filename="package://rover_gida/meshes/Rueda_6.STL" />
       </geometry>
     </collision>
@@ -1070,5 +1070,5 @@
   <!-- SENSOR KINECT -->
   <xacro:if value="$(arg kinect_enable)">
-    <xacro:include filename="$(find rover_rycsv)/urdf/kinect.gazebo.xacro" />
+    <xacro:include filename="$(find rover_gida)/urdf/kinect.gazebo.xacro" />
     <link name="Sensor_kinect">
       <inertial>
@@ -1092,5 +1092,5 @@
         <geometry>
           <mesh
-            filename="package://rover_rycsv/meshes/sensor_kinect.stl"
+            filename="package://rover_gida/meshes/sensor_kinect.stl"
             scale= "0.01 0.01 0.01"/>
         </geometry>
@@ -1107,5 +1107,5 @@
         <geometry>
           <mesh
-            filename="package://rover_rycsv/meshes/sensor_kinect.stl"
+            filename="package://rover_gida/meshes/sensor_kinect.stl"
             scale= "0.01 0.01 0.01"/>
         </geometry>
@@ -1140,6 +1140,6 @@
   <!-- CAMARA Y LIDAR -->
   <xacro:if value="$(arg camera_and_lidar_enable)">
-    <xacro:include filename="$(find rover_rycsv)/urdf/camera.gazebo.xacro" />
-    <xacro:include filename="$(find rover_rycsv)/urdf/lidar.gazebo.xacro" />
+    <xacro:include filename="$(find rover_gida)/urdf/camera.gazebo.xacro" />
+    <xacro:include filename="$(find rover_gida)/urdf/lidar.gazebo.xacro" />
     <link name="Camera">
       <inertial>
@@ -1202,5 +1202,5 @@
         <origin xyz="0 0 0" rpy="0 0 0"/>
         <geometry>
-          <mesh filename="package://rover_rycsv/meshes/hokuyo.dae"/>
+          <mesh filename="package://rover_gida/meshes/hokuyo.dae"/>
         </geometry>
       </visual>
@@ -1227,5 +1227,5 @@
   <!-- SENSOR IMU -->
   <xacro:if value="$(arg imu_enable)">
-    <xacro:include filename="$(find rover_rycsv)/urdf/imu.gazebo.xacro" />
+    <xacro:include filename="$(find rover_gida)/urdf/imu.gazebo.xacro" />
     <link name="IMU">
       <inertial>
@@ -1280,5 +1280,5 @@
   </xacro:if>
   <xacro:if value="$(arg gps_enable)">
-    <xacro:include filename="$(find rover_rycsv)/urdf/gps.gazebo.xacro" />
+    <xacro:include filename="$(find rover_gida)/urdf/gps.gazebo.xacro" />
     <link name="GPS">
       <inertial>

Commit message: Cambios menores

File: Proyecto/rover_rycsv/urdf/rover.urdf.xacro (robot description, xacro)
@@ -1,4 +1,4 @@
 <?xml version="1.0" encoding="utf-8"?>
-<robot name="rover_gida" xmlns:xacro="http://ros.org/wiki/xacro">
+<robot name="rover_rycsv" xmlns:xacro="http://ros.org/wiki/xacro">
   <xacro:arg name="imu_enable" default="true"/>
   <xacro:arg name="gps_enable" default="true"/>
@@ -29,5 +29,5 @@
       <geometry>
         <mesh
-          filename="package://rover_gida/meshes/Caja.STL" />
+          filename="package://rover_rycsv/meshes/Caja.STL" />
       </geometry>
       <material
@@ -81,5 +81,5 @@
       <geometry>
         <mesh
-          filename="package://rover_gida/meshes/Rocker_izq.STL" />
+          filename="package://rover_rycsv/meshes/Rocker_izq.STL" />
       </geometry>
       <material
@@ -135,5 +135,5 @@
       <geometry>
         <mesh
-          filename="package://rover_gida/meshes/Bogie_izq.STL" />
+          filename="package://rover_rycsv/meshes/Bogie_izq.STL" />
       </geometry>
       <material
@@ -189,5 +189,5 @@
       <geometry>
         <mesh
-          filename="package://rover_gida/meshes/Acople_1.STL" />
+          filename="package://rover_rycsv/meshes/Acople_1.STL" />
       </geometry>
       <material
@@ -243,5 +243,5 @@
       <geometry>
         <mesh
-          filename="package://rover_gida/meshes/Rueda_1.STL" />
+          filename="package://rover_rycsv/meshes/Rueda_1.STL" />
       </geometry>
       <material
@@ -257,5 +257,5 @@
       <geometry>
         <mesh
-          filename="package://rover_gida/meshes/Rueda_1.STL" />
+          filename="package://rover_rycsv/meshes/Rueda_1.STL" />
       </geometry>
     </collision>
@@ -299,5 +299,5 @@
       <geometry>
         <mesh
-          filename="package://rover_gida/meshes/Acople_2.STL" />
+          filename="package://rover_rycsv/meshes/Acople_2.STL" />
       </geometry>
       <material
@@ -351,5 +351,5 @@
       <geometry>
         <mesh
-          filename="package://rover_gida/meshes/Rueda_2.STL" />
+          filename="package://rover_rycsv/meshes/Rueda_2.STL" />
       </geometry>
       <material
@@ -365,5 +365,5 @@
       <geometry>
         <mesh
-          filename="package://rover_gida/meshes/Rueda_2.STL" />
+          filename="package://rover_rycsv/meshes/Rueda_2.STL" />
       </geometry>
     </collision>
@@ -407,5 +407,5 @@
       <geometry>
         <mesh
-          filename="package://rover_gida/meshes/Acople_3.STL" />
+          filename="package://rover_rycsv/meshes/Acople_3.STL" />
       </geometry>
       <material
@@ -461,5 +461,5 @@
       <geometry>
         <mesh
-          filename="package://rover_gida/meshes/Rueda_3.STL" />
+          filename="package://rover_rycsv/meshes/Rueda_3.STL" />
       </geometry>
       <material
@@ -475,5 +475,5 @@
       <geometry>
         <mesh
-          filename="package://rover_gida/meshes/Rueda_3.STL" />
+          filename="package://rover_rycsv/meshes/Rueda_3.STL" />
       </geometry>
     </collision>
@@ -517,5 +517,5 @@
       <geometry>
         <mesh
-          filename="package://rover_gida/meshes/Rocker_der.STL" />
+          filename="package://rover_rycsv/meshes/Rocker_der.STL" />
       </geometry>
       <material
@@ -571,5 +571,5 @@
       <geometry>
         <mesh
-          filename="package://rover_gida/meshes/Bogie_der.STL" />
+          filename="package://rover_rycsv/meshes/Bogie_der.STL" />
       </geometry>
       <material
@@ -625,5 +625,5 @@
       <geometry>
         <mesh
-          filename="package://rover_gida/meshes/Acople_4.STL" />
+          filename="package://rover_rycsv/meshes/Acople_4.STL" />
       </geometry>
       <material
@@ -679,5 +679,5 @@
       <geometry>
         <mesh
-          filename="package://rover_gida/meshes/Rueda_4.STL" />
+          filename="package://rover_rycsv/meshes/Rueda_4.STL" />
       </geometry>
       <material
@@ -693,5 +693,5 @@
       <geometry>
         <mesh
-          filename="package://rover_gida/meshes/Rueda_4.STL" />
+          filename="package://rover_rycsv/meshes/Rueda_4.STL" />
       </geometry>
     </collision>
@@ -735,5 +735,5 @@
       <geometry>
         <mesh
-          filename="package://rover_gida/meshes/Acople_5.STL" />
+          filename="package://rover_rycsv/meshes/Acople_5.STL" />
       </geometry>
       <material
@@ -787,5 +787,5 @@
       <geometry>
         <mesh
-          filename="package://rover_gida/meshes/Rueda_5.STL" />
+          filename="package://rover_rycsv/meshes/Rueda_5.STL" />
       </geometry>
       <material
@@ -801,5 +801,5 @@
       <geometry>
         <mesh
-          filename="package://rover_gida/meshes/Rueda_5.STL" />
+          filename="package://rover_rycsv/meshes/Rueda_5.STL" />
       </geometry>
     </collision>
@@ -843,5 +843,5 @@
       <geometry>
         <mesh
-          filename="package://rover_gida/meshes/Acople_6.STL" />
+          filename="package://rover_rycsv/meshes/Acople_6.STL" />
       </geometry>
       <material
@@ -897,5 +897,5 @@
       <geometry>
         <mesh
-          filename="package://rover_gida/meshes/Rueda_6.STL" />
+          filename="package://rover_rycsv/meshes/Rueda_6.STL" />
       </geometry>
       <material
@@ -911,5 +911,5 @@
       <geometry>
         <mesh
-          filename="package://rover_gida/meshes/Rueda_6.STL" />
+          filename="package://rover_rycsv/meshes/Rueda_6.STL" />
       </geometry>
     </collision>
@@ -1070,5 +1070,5 @@
   <!-- SENSOR KINECT -->
   <xacro:if value="$(arg kinect_enable)">
-    <xacro:include filename="$(find rover_gida)/urdf/kinect.gazebo.xacro" />
+    <xacro:include filename="$(find rover_rycsv)/urdf/kinect.gazebo.xacro" />
     <link name="Sensor_kinect">
       <inertial>
@@ -1092,5 +1092,5 @@
         <geometry>
           <mesh
-            filename="package://rover_gida/meshes/sensor_kinect.stl"
+            filename="package://rover_rycsv/meshes/sensor_kinect.stl"
             scale= "0.01 0.01 0.01"/>
         </geometry>
@@ -1107,5 +1107,5 @@
         <geometry>
           <mesh
-            filename="package://rover_gida/meshes/sensor_kinect.stl"
+            filename="package://rover_rycsv/meshes/sensor_kinect.stl"
             scale= "0.01 0.01 0.01"/>
         </geometry>
@@ -1140,6 +1140,6 @@
   <!-- CAMARA Y LIDAR -->
   <xacro:if value="$(arg camera_and_lidar_enable)">
-    <xacro:include filename="$(find rover_gida)/urdf/camera.gazebo.xacro" />
-    <xacro:include filename="$(find rover_gida)/urdf/lidar.gazebo.xacro" />
+    <xacro:include filename="$(find rover_rycsv)/urdf/camera.gazebo.xacro" />
+    <xacro:include filename="$(find rover_rycsv)/urdf/lidar.gazebo.xacro" />
     <link name="Camera">
       <inertial>
@@ -1202,5 +1202,5 @@
         <origin xyz="0 0 0" rpy="0 0 0"/>
         <geometry>
-          <mesh filename="package://rover_gida/meshes/hokuyo.dae"/>
+          <mesh filename="package://rover_rycsv/meshes/hokuyo.dae"/>
         </geometry>
       </visual>
@@ -1227,5 +1227,5 @@
   <!-- SENSOR IMU -->
   <xacro:if value="$(arg imu_enable)">
-    <xacro:include filename="$(find rover_gida)/urdf/imu.gazebo.xacro" />
+    <xacro:include filename="$(find rover_rycsv)/urdf/imu.gazebo.xacro" />
     <link name="IMU">
       <inertial>
@@ -1280,5 +1280,5 @@
   </xacro:if>
   <xacro:if value="$(arg gps_enable)">
-    <xacro:include filename="$(find rover_gida)/urdf/gps.gazebo.xacro" />
+    <xacro:include filename="$(find rover_rycsv)/urdf/gps.gazebo.xacro" />
     <link name="GPS">
       <inertial>
